File: KiCad-project/obi1/Flash_Memory.sch (KiCad schematic (older format))
At the start: 8 parts, among them IC3 FLASH

Commit message: Routear
Parts:
- renumbered C53 to C54, C54 to C55, R44 to R45, R45 to R46, R46 to R47, R47 to R48, R48 to R49
Changed lines of the file:
@@
 $EndComp
 $Comp
-L Device:R R46
+L Device:R R47
 U 1 1 5D98FC5E
 P 2300 1800
-F 0 "R46" H 2370 1846 50  0000 L CNN
+F 0 "R47" H 2370 1846 50  0000 L CNN
 F 1 "@2.4K;1/4W;0805;1%" H 1400 1800 50  0000 L CNN
 F 2 "Resistor_SMD:R_0805_2012Metric_Pad1.20x1.40mm_HandSolder" V 2230 1800 50  0001 C CNN
@@
 $EndComp
 $Comp
-L Device:R R45
+L Device:R R46
 U 1 1 5D9902C5
 P 1950 2050
-F 0 "R45" V 1950 2050 50  0000 C CNN
+F 0 "R46" V 1950 2050 50  0000 C CNN
 F 1 "@100;1/4W;0805;1%" V 1900 1550 50  0000 C CNN
 F 2 "Resistor_SMD:R_0805_2012Metric_Pad1.20x1.40mm_HandSolder" V 1880 2050 50  0001 C CNN
@@
 $EndComp
 $Comp
-L Device:R R44
+L Device:R R45
 U 1 1 5D990C48
 P 1700 2150
-F 0 "R44" V 1700 2150 50  0000 C CNN
+F 0 "R45" V 1700 2150 50  0000 C CNN
 F 1 "@100;1/4W;0805;1%" V 1800 2150 50  0000 C CNN
 F 2 "Resistor_SMD:R_0805_2012Metric_Pad1.20x1.40mm_HandSolder" V 1630 2150 50  0001 C CNN
@@
 $EndComp
 $Comp
-L Device:R R47
+L Device:R R48
 U 1 1 5D99165B
 P 4450 2050
-F 0 "R47" V 4450 2050 50  0000 C CNN
+F 0 "R48" V 4450 2050 50  0000 C CNN
 F 1 "@100;1/4W;0805;1%" V 4350 2150 50  0000 C CNN
 F 2 "Resistor_SMD:R_0805_2012Metric_Pad1.20x1.40mm_HandSolder" V 4380 2050 50  0001 C CNN
@@
 	4200 1950 4200 1800
 $Comp
-L Device:R R48
+L Device:R R49
 U 1 1 5D991B6E
 P 4450 2250
-F 0 "R48" V 4450 2250 50  0000 C CNN
+F 0 "R49" V 4450 2250 50  0000 C CNN
 F 1 "@100;1/4W;0805;1%" V 4550 2250 50  0000 C CNN
 F 2 "Resistor_SMD:R_0805_2012Metric_Pad1.20x1.40mm_HandSolder" V 4380 2250 50  0001 C CNN
@@
 XC_T3
 $Comp
-L Device:C C53
+L Device:C C54
 U 1 1 5DAEFC38
 P 4350 1650
-F 0 "C53" H 4500 1700 50  0000 L CNN
+F 0 "C54" H 4500 1700 50  0000 L CNN
 F 1 "@0.47uF;6.3V;X5R;0402;10%" H 3850 1750 50  0000 L CNN
 F 2 "Capacitor_SMD:C_0402_1005Metric_Pad0.74x0.62mm_HandSolder" H 4388 1500 50  0001 C CNN
@@
 $EndComp
 $Comp
-L Device:C C54
+L Device:C C55
 U 1 1 5DAF0967
 P 4900 1650
-F 0 "C54" H 5050 1700 50  0000 L CNN
+F 0 "C55" H 5050 1700 50  0000 L CNN
 F 1 "@4.7uF;6.3V;X5R;0805;10%" H 4750 1550 50  0000 L CNN
 F 2 "Capacitor_SMD:C_0805_2012Metric_Pad1.18x1.45mm_HandSolder" H 4938 1500 50  0001 C CNN
