File: KiCad-project/obi1/Inputs_Outputs.sch (KiCad schematic (older format))
At the start: 47 parts, among them J5 Conn_01x10, J6 Conn_01x10, J7 Conn_02x17_Counter_Clockwise, J8 Conn_02x11_Counter_Clockwise, SW3 SW_DIP_x08, U7 RV1, U8 RV2

Commit message: Routear
Parts:
- renumbered C45 to C46, C46 to C47, C47 to C48, C48 to C49, C49 to C50, C50 to C51, C51 to C52, C52 to C53, R20 to R21, R21 to R22, R22 to R23, R23 to R24, R24 to R25, R25 to R26, R26 to R27, R27 to R28, R28 to R29, R29 to R30, R30 to R31, R31 to R32, R32 to R33, R33 to R34, R34 to R35, R35 to R36, R36 to R37, R37 to R38, R38 to R39, R39 to R40, R40 to R41, R41 to R42, R42 to R43, R43 to R44

Commit message: Resize board, change layout, re-route IO pins, new imu added
Connections:
- net IO_C00 is gone; now on net IO_A02: J8.3 (Pin_3)
- net IO_F00 is gone; now on net IO_E03: J7.23 (Pin_23)
- net IO_G00 is gone; now on net IO_E04: J7.24 (Pin_24)
- net IO_G01 is gone; now on net IO_E07: J7.27 (Pin_27)
- net IO_G02 is gone; now on net IO_F01: J7.28 (Pin_28)
- net IO_G03 is gone; now on net IO_D04: J7.11 (Pin_11)
- net IO_G04 is gone; now on net IO_D07: J7.14 (Pin_14)
- net IO_H01 is gone; now on net IO_E01: J7.21 (Pin_21)
- net IO_H03 is gone; now on net IO_D02: J7.9 (Pin_9)
- net IO_H04 is gone; now on net IO_D05: J7.12 (Pin_12)
- net IO_H06 is gone; now on net IO_E02: J7.22 (Pin_22)
- net IO_H07 is gone; now on net IO_C07: J7.7 (Pin_7)
- net IO_I00 is gone; now on net IO_D03: J7.10 (Pin_10)
- net IO_I01 is gone; now on net IO_D06: J7.13 (Pin_13)
- net IO_I02 is gone; now on net IO_D01: J7.8 (Pin_8)
- net IO_I05 is gone; now on net IO_C06: J7.6 (Pin_6)
- net IO_I06 is gone; now on net IO_C05: J7.5 (Pin_5)
- net +3V3: now also J7.15 (Pin_15), J7.16 (Pin_16), J8.10 (Pin_10), J8.9 (Pin_9); no longer J7.19 (Pin_19), J7.20 (Pin_20)
- net +5V: now also J7.19 (Pin_19), J7.20 (Pin_20), J8.13 (Pin_13), J8.14 (Pin_14); no longer J7.15 (Pin_15), J7.16 (Pin_16)
- net DS_2_XC1: now also R29.1; no longer J8.4 (Pin_4)
- net DS_2_XC2: now also R30.1; no longer J8.6 (Pin_6)
- net DS_2_XC3: now also R31.1
- net DS_2_XC4: now also R32.1; no longer J8.7 (Pin_7)
- net DS_2_XC5: now also R33.1; no longer J8.9 (Pin_9)
- net DS_2_XC6: now also R34.1; no longer J8.8 (Pin_8)
- net DS_2_XC7: now also R35.1; no longer J8.15 (Pin_15)
- net DS_2_XC8: now also R36.1
- net GND: now also J8.11 (Pin_11), J8.12 (Pin_12); no longer J8.1 (Pin_1), J8.2 (Pin_2)
- net IO_A00: now also J8.1 (Pin_1)
- net IO_A01: now also J8.2 (Pin_2); no longer J8.17 (Pin_17)
- net IO_A02: no longer J8.16 (Pin_16)
- net IO_A03: now also J8.4 (Pin_4); no longer J8.18 (Pin_18)
- net IO_A04: now also J8.5 (Pin_5); no longer R33.1
- net IO_A05: now also J8.6 (Pin_6)
- net IO_A06: now also J8.7 (Pin_7); no longer J8.19 (Pin_19)
- net IO_A07: now also J8.8 (Pin_8); no longer R32.1
- net IO_B00: now also J8.15 (Pin_15); no longer R34.1
- net IO_B01: now also J8.16 (Pin_16); no longer J8.20 (Pin_20)
- net IO_B02: now also J8.17 (Pin_17); no longer J8.22 (Pin_22)
- net IO_B03: now also J8.18 (Pin_18); no longer R29.1
- net IO_B04: now also J8.19 (Pin_19); no longer J7.33 (Pin_33)
- net IO_B05: now also J8.20 (Pin_20); no longer R30.1
- net IO_B07: now also J8.22 (Pin_22); no longer J7.34 (Pin_34)
- net IO_C01: now also J7.1 (Pin_1); no longer J8.5 (Pin_5)
- net IO_C02: now also J7.2 (Pin_2); no longer J7.1 (Pin_1)
- net IO_C03: now also J7.3 (Pin_3); no longer J7.4 (Pin_4)
- net IO_C04: now also J7.4 (Pin_4); no longer J7.2 (Pin_2)
- net IO_C06: no longer J7.3 (Pin_3)
- net IO_D01: no longer R35.1
- net IO_D02: no longer J7.31 (Pin_31)
- net IO_D04: no longer R31.1
- net IO_D05: no longer R36.1
- net IO_E01: no longer J8.14 (Pin_14)
- net IO_E02: no longer J8.11 (Pin_11)
- net IO_E04: no longer J8.10 (Pin_10)
- net IO_E05: now also J7.25 (Pin_25); no longer J8.13 (Pin_13)
- net IO_E06: now also J7.26 (Pin_26); no longer J8.12 (Pin_12)
- net IO_E07: no longer J7.25 (Pin_25)
- net IO_F01: no longer J7.32 (Pin_32)
- net IO_F03: now also J7.30 (Pin_30)
- net IO_F04: now also J7.31 (Pin_31)
- net IO_F05: now also J7.32 (Pin_32)
- net IO_F06: now also J7.33 (Pin_33); no longer J7.30 (Pin_30)
- net IO_F07: now also J7.34 (Pin_34); no longer J7.26 (Pin_26)
- no-connect marks 29 -> 0
