File: KiCad-project/obi1/POWER_SUPLY.sch (KiCad schematic (older format))
At the start: 9 parts, among them J1 USB, U1 RG3V3, U2 REG1V2

Commit message: Changed RAM by Cypres Model -rebuild symbolic and changed footprint
Parts:
- J1: footprint egalan_lib:101181930001LF -> egalan:101181930001LF
- U1: footprint egalan_lib:SOT230P700X180-4N3.3 -> egalan:SOT230P700X180-4N3.3
- U2: footprint egalan_lib:SOT230P700X180-4N1.2 -> egalan:SOT230P700X180-4N1.2
Changed lines of the file:
@@
 F 0 "U1" H 6050 3115 50  0000 C CNN
 F 1 "RG3V3" H 6050 3024 50  0000 C CNN
-F 2 "egalan_lib:SOT230P700X180-4N3.3" H 5650 2350 50  0001 L BNN
+F 2 "egalan:SOT230P700X180-4N3.3" H 5650 2350 50  0001 L BNN
 F 3 "" H 5700 2250 50  0001 L BNN
 F 4 "AZ1117EH-3.3TRG1" H 5750 2450 50  0001 L BNN "Field4"
@@
 F 0 "U2" H 6050 3965 50  0000 C CNN
 F 1 "REG1V2" H 6050 3874 50  0000 C CNN
-F 2 "egalan_lib:SOT230P700X180-4N1.2" H 5650 3200 50  0001 L BNN
+F 2 "egalan:SOT230P700X180-4N1.2" H 5650 3200 50  0001 L BNN
 F 3 "" H 5700 3100 50  0001 L BNN
 	1    6050 3600
@@
 F 0 "J1" H 5000 3300 50  0000 C CNN
 F 1 "USB" H 5000 3200 50  0000 C CNN
-F 2 "egalan_lib:101181930001LF" H 5350 3100 50  0001 L CNN
+F 2 "egalan:101181930001LF" H 5350 3100 50  0001 L CNN
 F 3 "" H 7450 2200 50  0001 L CNN
 	1    4500 3000
