File: KiCad-project/obi1/obi1.kicad_pcb (KiCad board)
At the start: 4 copper layers, 78.7 x 86.4 mm, 138 parts, among them IC2 DAC, IC3 FLASH, J1 USB, J2 JTAG-H, J3 Conn_01x04, J4 Conn_01x04, J5 Conn_01x10, J6 Conn_01x10, J7 Conn_02x17_Counter_Clockwise, J8 Conn_02x11_Counter_Clockwise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

Commit message: IMU changed again, Final IMU= LSM6DSMTR, First Order to OSHPark
Parts:
- removed C43: @1uF;6.3V;X5R;0805;10%, Capacitor_SMD:C_0805_2012Metric_Pad1.18x1.45mm_HandSolder
- removed C44: @0.12uF;10V;X7R;0603;10%, Capacitor_SMD:C_0603_1608Metric_Pad1.08x0.95mm_HandSolder
- removed C45: @6800pF;10V;X7R;0603;10%, Capacitor_SMD:C_0603_1608Metric_Pad1.08x0.95mm_HandSolder
- removed R19: @10;1/4W;0805;1%, Resistor_SMD:R_0805_2012Metric_Pad1.20x1.40mm_HandSolder
- removed R20: @10K;1/4W;0805;1%, Resistor_SMD:R_0805_2012Metric_Pad1.20x1.40mm_HandSolder
- C42: value @1uF;6.3V;X5R;0805;10% -> @0.1uF;6.3V;X5R;0805;10%; moved to F.Cu
- J1: footprint egalan_lib:101181930001LF -> egalan:101181930001LF
- U1: footprint egalan_lib:SOT230P700X180-4N3.3 -> egalan:SOT230P700X180-4N3.3
- U2: footprint egalan_lib:SOT230P700X180-4N1.2 -> egalan:SOT230P700X180-4N1.2
- U6: value BMF055 -> LSM6DSMTR; footprint Package_LGA:LGA-28_5.2x3.8mm_P0.5mm -> egalan:PQFN50P300X250X86-14N
- moved C41 9.09 mm to (177.9, 99.5)
- moved C42 3.37 mm to (181.9, 98.4), turned to 270 degrees
- moved J1 2.03 mm to (121.2, 76.2)
- moved U6 2.00 mm to (177.6, 95.6), turned to 0 degrees
Connections:
- C42 pad 1: Net-(C42-Pad1) -> +3V3
- U3 pad C16: IMU_PB03 -> IMU_INT2
- U3 pad D16: IMU_PB02 -> IMU_CS
- U3 pad E13: nReset -> (no net)
- U3 pad E16: IMU_PB01 -> IMU_SCL_SPC
- U3 pad F12: IMU_PA17 -> (no net)
- U3 pad F14: IMU_SCX -> (no net)
- U3 pad F15: IMU_PB00 -> IMU_SDA_SDI_SDO
- U3 pad G11: IMU_PA16 -> (no net)
- U3 pad G14: IMU_PA30 -> IMU_INT1
- U3 pad G16: IMU_PA31 -> IMU_SDO_SAO
- U3 pad H11: IMU_PA18 -> (no net)
- U3 pad H13: IMU_PA20 -> (no net)
- U3 pad H14: IMU_PB17 -> (no net)
- U3 pad H15: IMU_PA27 -> (no net)
- U3 pad H16: IMU_PA28 -> (no net)
- U3 pad J12: IMU_PA23 -> (no net)
- U3 pad J14: IMU_PA24 -> (no net)
- U3 pad J16: IMU_PB23 -> (no net)
- U3 pad K14: IMU_PA19 -> (no net)
- U3 pad K15: IMU_PA21 -> (no net)
- U3 pad K16: IMU_PA22 -> (no net)
- U3 pad L10: (no net) -> IO_B00
- U3 pad L14: IMU_PB16 -> (no net)
- U3 pad N11: (no net) -> GND
- U3 pad T11: IO_B00 -> +3V3
- U6 pad 1: IMU_PB03 -> IMU_SDO_SAO
- U6 pad 10: IMU_PA28 -> (no net)
- U6 pad 11: Net-(C42-Pad1) -> (no net)
- U6 pad 12: IMU_PA27 -> IMU_CS
- U6 pad 13: IMU_PB23 -> IMU_SCL_SPC
- U6 pad 14: IMU_PA24 -> IMU_SDA_SDI_SDO
- U6 pad 3: +3V3 -> GND
- U6 pad 4: IMU_PB02 -> IMU_INT1
- U6 pad 5: IMU_PB01 -> +3V3
- U6 pad 6: IMU_PB00 -> GND
- U6 pad 7: IMU_PA31 -> GND
- U6 pad 8: IMU_PA30 -> +3V3
- U6 pad 9: Net-(C43-Pad1) -> IMU_INT2
Routing:
- net +5V: track 213.3 -> 257.8 mm, vias 7 -> 6
- net nReset: track 20.8 -> 0.00 mm, vias 1 -> 0
- net IMU_INT2: track 0.00 -> 17.6 mm
- net IMU_PA16: track 16.5 -> 0.00 mm, vias 3 -> 0
- net IMU_PA18: track 16.4 -> 0.00 mm, vias 2 -> 0
- net IMU_PB03: track 15.1 -> 0.00 mm
- net Net-(C42-Pad1): track 15.1 -> 0.00 mm, vias 1 -> 0
- net IMU_PA17: track 15.0 -> 0.00 mm, vias 2 -> 0
- net IMU_PA19: track 14.2 -> 0.00 mm, vias 2 -> 0
- net IMU_SCX: track 12.8 -> 0.00 mm, vias 2 -> 0
- net IMU_PA20: track 12.7 -> 0.00 mm, vias 2 -> 0
- net IMU_PB16: track 12.7 -> 0.00 mm, vias 2 -> 0
- net IMU_PB17: track 12.6 -> 0.00 mm, vias 2 -> 0
- net IMU_CS: track 0.00 -> 12.5 mm
- net IMU_INT1: track 0.00 -> 11.7 mm
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Other:
- net class 5v added: clearance 0.1524, trace_width 2.032, via_dia 0.4, via_drill 0.2
